File: hello/hello.kicad_sch (KiCad schematic)
At the start: 12 parts, among them J1 pwm, J2 voltmeter, J3 common, J4 continuous, J5 common, SW1 SW_SPST, U1 Arduino nano, U2 oled i2c, U3 Rotary Encoder

Commit message: final pcb
Parts:
- removed SW1: SW_SPST, symbol Switch:SW_SPST
- added SW1: SW_SPST, SPST:JUDCOSPST, symbol Switch2:SW_SPST
- BT1: footprint (none) -> Battery:BatteryHolder_Keystone_2479_3xAAA
- J1, J2, J3, J4, J5: footprint (none) -> Connector_PinSocket_1.27mm:PinSocket_1x01_P1.27mm_Vertical
- R1: footprint (none) -> Resistor_THT:R_Axial_DIN0204_L3.6mm_D1.6mm_P1.90mm_Vertical
- R2: footprint (none) -> Connector_PinSocket_1.27mm:PinSocket_1x02_P1.27mm_Vertical
- U1: footprint (none) -> MCU_arduino_nano:Arduino_nano
- U2: footprint (none) -> Connector_PinSocket_1.27mm:PinSocket_1x04_P1.27mm_Vertical
- U3: footprint (none) -> Connector_PinSocket_1.27mm:PinSocket_1x05_P1.27mm_Vertical
Connections:
- net +5V: now also U2.2 (VCC), U3.2 (VCC); no longer U2. (VCC), U3. (VCC)
- net CLK: now also U3.5 (CLK); no longer U3. (VCC)
- net DT: now also U3.4 (DT); no longer U3. (VCC)
- net GND: now also U2.1 (GND), U3.1 (GND), SW1.T (A); no longer U2. (VCC), U3. (VCC)
- net SCL: now also U2.3 (SCL); no longer U2. (VCC)
- net SDA: now also U2.4 (SDA); no longer U2. (VCC)
- net switch: now reaches BT1.2 (-)
- net switch: now also SW1.P (B)
